Commit message: urdf

File: robot/franka_description/robot.urdf (robot description, URDF)
Before this commit: robot fr3, 14 links, 13 joints
Links:
- link fr3_leftfinger: geometry collision mesh filename=meshes/collision/finger.obj; visual mesh filename=meshes/visual/finger.obj
- link fr3_rightfinger: geometry collision mesh filename=meshes/collision/finger.obj; visual mesh filename=meshes/visual/finger.obj
